File: pcbs/control/control.kicad_pcb (KiCad board)
At the start: 2 copper layers, 93.8 x 39.5 mm, 58 parts, among them J2 USB4125-GF-A-0190, J3 Conn_01x10_Pin, J4 Conn_02x04_Odd_Even, Q1 SI2393DS-T1-GE3, Q10 DMN2020LSN-7, Q2 SI2393DS-T1-GE3, Q3 SI2393DS-T1-GE3, Q4 SI2393DS-T1-GE3, Q5 DMN2020LSN-7, Q6 DMN2020LSN-7, Q7 DMN2020LSN-7, Q8 DMN2020LSN-7, Q9 DMN2020LSN-7, SW1 Sparkle, SW2 Time Adj, U1 DS18B20U, U2 DS3231MZ, U3 TPS259621DDAT, U6 ATmega328PB-A

Commit message: pcb and enclosure update
Parts:
- removed BT1: 3000TR, Clock:BAT_3000TR
- added J1: Conn_01x02_Pin, Connector_JST:JST_PH_S2B-PH-SM4-TB_1x02-1MP_P2.00mm_Horizontal, B.Cu at (-18.5, 3.62)
- F1, F2, F3, F4, F5, F6: value Fuse -> 0.375 A
- Q1, Q2, Q3, Q4: value SI2393DS-T1-GE3 -> PMV35EPER
- SW1: value Sparkle -> Sparkle Btn
- SW2: value Time Adj -> Time Adj Btn
- U3: value TPS259621DDAT -> TPS259620
Routing:
- net /RTC_BAT: track 40.5 -> 27.9 mm
- net GNDD: vias 14 -> 13
Other:
- outline, holes or cut-outs redrawn

Commit message: lengthened display cable
Parts:
- moved J1 40.6 mm to (21.3, 12.1), turned to 0 degrees
Connections:
- J1 pad 1: GNDD -> /RTC_BAT
- J1 pad 2: /RTC_BAT -> GNDD
Routing:
- net /PIN 20: track 24.0 -> 26.6 mm
- net /RTC_BAT: track 27.9 -> 29.9 mm, vias 1 -> 3

Commit message: rv-3028 board
Parts:
- removed the C4 at (-20.0, -9.71)
- removed the J1 at (21.3, 12.1)
- removed the R19 at (-29.4, -4.20)
- removed the R21 at (-26.4, -1.89)
- removed the R22 at (-18.4, -6.83)
- removed the U3 at (-23.9, -5.80)
- added C2: 1uF, Capacitor_SMD:C_0805_2012Metric, F.Cu at (-23.5, -0.25)
- added C8: FC0V224ZFTBR24, Clock:CAPAE1080X550N, B.Cu at (-14.8, 3.50)
- added C9: FC0V224ZFTBR24, Clock:CAPAE1080X550N, B.Cu at (3.00, 3.50)
- added IC1: TPS25944LRVCR, Clock:QFN50P300X400X80-21N, F.Cu at (-22.2, -4.75)
- added R3: 56.2k, Resistor_SMD:R_0805_2012Metric, F.Cu at (-23.5, -8.50)
- added R4: 24.9k, Resistor_SMD:R_0805_2012Metric, F.Cu at (-19.8, -8.50)
- added R5: 8.45k, Resistor_SMD:R_0805_2012Metric, F.Cu at (-19.0, -5.25)
- added R6: 110k, Resistor_SMD:R_0805_2012Metric, F.Cu at (-19.0, -1.75)
- C1: value 1uF -> 0.1uF
- D1: value LED -> Status LED (Amber)
- F1, F2, F3, F4, F5, F6: value 0.375 A -> 375 mA
- R9: renamed from R18; value 60 -> 300
- U2: value DS3231MZ -> RV-3028-C7_32.768KHZ_1PPM-TA-QC; footprint Package_SO:SOIC-8_3.9x4.9mm_P1.27mm -> Clock:IC_RV-3028-C7_32.768KHZ_1PPM-TA-QC
- moved C1 9.90 mm to (-21.0, -0.25), turned to 90 degrees
- moved R10 7.08 mm to (5.25, 0.00)
- moved C6 5.85 mm to (33.0, -3.00), turned to 49 degrees
- moved C7 4.79 mm to (-3.25, 0.00)
- moved R11 4.76 mm to (3.00, 0.00)
- moved R2 1.20 mm to (0.00, -11.5)
- moved R1 0.92 mm to (3.50, -11.5), turned to 180 degrees
- moved R23 0.55 mm to (38.2, 4.25)
- moved C5 0.35 mm to (9.50, -3.00)
- moved R9 0.32 mm to (20.0, -12.8), turned to 180 degrees
- moved Q1 0.25 mm to (-14.2, 7.00)
- moved R22 0.24 mm to (26.0, -9.00)
- moved D1 0.22 mm to (20.0, -10.5)
- moved C3 0.14 mm to (-11.0, -2.00)
- moved J3 0.12 mm to (38.2, 6.50)
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- renumbered C6 to C3, C5 to C4, C8 to C5, C3 to C6, C2 to C7, J3 to J1, J4 to J3, Q6 to Q10, Q10 to Q6, Q9 to Q7, Q7 to Q9, R15 to R1, R11 to R10, R12 to R11, R1 to R12, R2 to R13, R3 to R14, R4 to R15, R5 to R16, R10 to R17, R9 to R18, R8 to R19, R16 to R2, R7 to R20, R6 to R21, R20 to R22, R17 to R23, R14 to R7, R13 to R8, U6 to U1, D5 to U3, U1 to U4
Connections:
- C1 pad 2: /5v -> /VBUS
- R9 pad 1: Net-(D1-A) -> /ADC2
- R9 pad 2: /ADC2 -> Net-(D1-A)
- U2 pad 2: /3.3v -> unconnected-(U2-~{INT}-Pad2)
- U2 pad 3: unconnected-(U2-~{INT}/SQW-Pad3) -> /SCL
- U2 pad 4: unconnected-(U2-~{RST}-Pad4) -> /SDA
- U2 pad 6: /RTC_BAT -> Net-(C8-+)
- U2 pad 7: /SDA -> /3.3v
- U2 pad 8: /SCL -> GNDD
Routing:
- net GNDD: track 13.3 -> 68.1 mm, vias 13 -> 25
- net /RTC_BAT: track 29.9 -> 0.00 mm, vias 3 -> 0
- net Net-(C8-+): track 0.00 -> 13.8 mm, vias 0 -> 1
- net /5v: track 69.3 -> 59.7 mm
- net /PIN 5: track 45.7 -> 36.5 mm
- net /VBUS: track 30.1 -> 37.7 mm
- net /PIN 6: track 53.3 -> 47.0 mm
- net /3.3v: track 155.0 -> 160.6 mm
- net /SDA: track 26.8 -> 22.2 mm
- net Net-(IC1-OVP): track 0.00 -> 4.58 mm
- net /SCL: track 26.6 -> 22.5 mm
- net Net-(IC1-EN): track 0.00 -> 3.84 mm
- net /PIN 9: track 43.0 -> 46.3 mm
- net /PIN 20: track 26.6 -> 23.6 mm
- net Net-(U3-EN/UVLO): track 2.80 -> 0.00 mm
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- added copper zone on In1.Cu, net GNDD
- added copper zone on In2.Cu, net GNDD
- removed copper zone on B.Cu, net GNDD
- removed copper zone on F.Cu, net GNDD
Other:
- outline, holes or cut-outs redrawn
- copper layers 2 -> 4
- board text added: "paper sunshine clock"
- board text added: "v1.1 Oct 2025"
- board text removed: "Paper Sunshine Clock v1 2024"
